Commit message: Add files via upload

File: ur_description/urdf/mobile_base_without_arm.urdf (robot description, URDF)
Before this commit: robot ur10, 7 links, 6 joints
Links:
- removed link world
- link base_link: mass 47.873 -> 147.873
- link front_left_wheel: mass 2.6578 -> 50.6578
- link front_right_wheel: mass 2.6578 -> 50.6578
- link rear_left_wheel: mass 2.6578 -> 50.6578
- link rear_right_wheel: mass 2.6578 -> 50.6578
Joints:
- removed joint world_joint
